Commit message: Add UR base adatper

File: robotiq_85_description/urdf/robotiq_85_gripper_macro.urdf.xacro (robot description, xacro)
@@ -2,5 +2,4 @@
 <robot name="robotiq_85_gripper" xmlns:xacro="http://ros.org/wiki/xacro">
 	<xacro:include filename="$(find robotiq_85_description)/urdf/robotiq_85_gripper.transmission.xacro" />
-	<xacro:property name="pi" value="3.14159"/>
 	<xacro:macro name="mimic_joint_plugin_gazebo" params="name_prefix parent_joint mimic_joint has_pid:=false multiplier:=1.0 offset:=0 sensitiveness:=0.0 max_effort:=1.0 robot_namespace:=''">
 		<gazebo>
@@ -28,4 +27,15 @@
 		</joint>
 		<link name="${prefix}robotiq_85_base_link">
+			<!-- Visual aid for grasping -->
+			<visual>
+				<origin xyz="0.16 0 0" rpy="0 0 0" />
+        <geometry>
+          <sphere radius="0.007"/>
+        </geometry>
+        <material name="">
+					<color rgba="0 1.0 0 1.0"/>
+        </material>
+      </visual>
+			<!-- Gripper body -->
 			<visual>
 				<geometry>

Commit message: cleanup tabs and whitespace

File: robotiq_85_description/urdf/robotiq_85_gripper_macro.urdf.xacro (robot description, xacro)
@@ -30,11 +30,11 @@
 			<visual>
 				<origin xyz="0.16 0 0" rpy="0 0 0" />
-        <geometry>
-          <sphere radius="0.007"/>
-        </geometry>
-        <material name="">
+				<geometry>
+					<sphere radius="0.007"/>
+				</geometry>
+				<material name="">
 					<color rgba="0 1.0 0 1.0"/>
-        </material>
-      </visual>
+				</material>
+			</visual>
 			<!-- Gripper body -->
 			<visual>

Commit message: Make ros_control optional (#9)
* Add argument to make ros_control optional
* Document ros_control xacro for simulation

File: robotiq_85_description/urdf/robotiq_85_gripper_macro.urdf.xacro (robot description, xacro)
@@ -20,9 +20,15 @@
 		</gazebo>
 	</xacro:macro>
-	<xacro:macro name="robotiq_85_gripper" params="prefix parent *origin">
-		<!-- ros2 control include -->
-		<xacro:include filename="$(find robotiq_85_description)/urdf/robotiq_85_gripper.ros2_control.xacro"/>
-		<!-- ros2 control instance -->
-		<xacro:robotiq_85_gripper_ros2_control name="RobotiqGripperSystem"/>
+	<xacro:macro name="robotiq_85_gripper" params="prefix parent *origin sim:=false">
+		<!-- The current hardware driver does not depend on ros2_control but we do utilize
+				 it for simulating the gripper in Gazebo. Enabling this on hardware causes the
+				 JointStateBroadcaster to publish values for all joints including ones that are
+				 mimic'd which is causing issues on systems consuming the joint_state data. -->
+		<xacro:if value="${sim}">
+			<!-- ros2 control include -->
+			<xacro:include filename="$(find robotiq_85_description)/urdf/robotiq_85_gripper.ros2_control.xacro"/>
+			<!-- ros2 control instance -->
+			<xacro:robotiq_85_gripper_ros2_control name="RobotiqGripperSystem"/>
+		</xacro:if>
 		<joint name="${prefix}robotiq_85_base_joint" type="fixed">
 			<parent link="${parent}"/>

Commit message: Removed sphere from gripper visualization

File: robotiq_85_description/urdf/robotiq_85_gripper_macro.urdf.xacro (robot description, xacro)
@@ -3,20 +3,20 @@
 	<xacro:include filename="$(find robotiq_85_description)/urdf/robotiq_85_gripper.transmission.xacro" />
 	<xacro:macro name="mimic_joint_plugin_gazebo" params="name_prefix parent_joint mimic_joint has_pid:=false multiplier:=1.0 offset:=0 sensitiveness:=0.0 max_effort:=1.0 robot_namespace:=''">
-		<gazebo>
-			<plugin name="${name_prefix}mimic_joint_plugin" filename="libroboticsgroup_gazebo_mimic_joint_plugin.so">
-				<joint>${parent_joint}</joint>
-				<mimicJoint>${mimic_joint}</mimicJoint>
-				<xacro:if value="${has_pid}">                     <!-- if set to true, PID parameters from "/gazebo_ros_control/pid_gains/${mimic_joint}" are loaded -->
-					<hasPID />
-				</xacro:if>
-				<multiplier>${multiplier}</multiplier>
-				<offset>${offset}</offset>
-				<sensitiveness>${sensitiveness}</sensitiveness>   <!-- if absolute difference between setpoint and process value is below this threshold, do nothing; 0.0 = disable [rad] -->
-				<maxEffort>${max_effort}</maxEffort>              <!-- only taken into account if has_pid:=true [Nm] -->
-				<xacro:unless value="${robot_namespace == ''}">
-					<robotNamespace>($robot_namespace)</robotNamespace>
-				</xacro:unless>
-			</plugin>
-		</gazebo>
+    <gazebo>
+      <plugin name="${name_prefix}mimic_joint_plugin" filename="libroboticsgroup_gazebo_mimic_joint_plugin.so">
+        <joint>${parent_joint}</joint>
+        <mimicJoint>${mimic_joint}</mimicJoint>
+        <xacro:if value="${has_pid}">                     <!-- if set to true, PID parameters from "/gazebo_ros_control/pid_gains/${mimic_joint}" are loaded -->
+          <hasPID />
+        </xacro:if>
+        <multiplier>${multiplier}</multiplier>
+        <offset>${offset}</offset>
+        <sensitiveness>${sensitiveness}</sensitiveness>   <!-- if absolute difference between setpoint and process value is below this threshold, do nothing; 0.0 = disable [rad] -->
+        <maxEffort>${max_effort}</maxEffort>              <!-- only taken into account if has_pid:=true [Nm] -->
+        <xacro:unless value="${robot_namespace == ''}">
+          <robotNamespace>($robot_namespace)</robotNamespace>
+        </xacro:unless>
+      </plugin>
+    </gazebo>
 	</xacro:macro>
 	<xacro:macro name="robotiq_85_gripper" params="prefix parent *origin sim:=false">
@@ -37,14 +37,4 @@
 		</joint>
 		<link name="${prefix}robotiq_85_base_link">
-			<!-- Visual aid for grasping -->
-			<visual>
-				<origin xyz="0.16 0 0" rpy="0 0 0" />
-				<geometry>
-					<sphere radius="0.007"/>
-				</geometry>
-				<material name="">
-					<color rgba="0 1.0 0 1.0"/>
-				</material>
-			</visual>
 			<!-- Gripper body -->
 			<visual>
@@ -101,7 +91,7 @@
 			<material>Gazebo/Grey</material>
 		</gazebo>
-		<xacro:mimic_joint_plugin_gazebo name_prefix="{prefix}robotiq_85_right_knuckle_joint"
+    <xacro:mimic_joint_plugin_gazebo name_prefix="{prefix}robotiq_85_right_knuckle_joint"
 			parent_joint="${prefix}robotiq_85_left_knuckle_joint" mimic_joint="${prefix}robotiq_85_right_knuckle_joint"
-			multiplier="1.0" max_effort="10.0" />
+      multiplier="1.0" max_effort="10.0" />
 		<link name="${prefix}robotiq_85_left_knuckle_link">
 			<visual>
@@ -198,7 +188,7 @@
 			<mimic joint="${prefix}robotiq_85_left_knuckle_joint" offset="0"/>
 		</joint>
-		<xacro:mimic_joint_plugin_gazebo name_prefix="${prefix}robotiq_85_left_inner_knuckle_joint"
+    <xacro:mimic_joint_plugin_gazebo name_prefix="${prefix}robotiq_85_left_inner_knuckle_joint"
 			parent_joint="${prefix}robotiq_85_left_knuckle_joint" mimic_joint="${prefix}robotiq_85_left_inner_knuckle_joint"
-			multiplier="1.0" max_effort="10.0" />
+      multiplier="1.0" max_effort="10.0" />
 		<joint name="${prefix}robotiq_85_right_inner_knuckle_joint" type="continuous">
 			<parent link="${prefix}robotiq_85_base_link"/>
@@ -209,7 +199,7 @@
 			<mimic joint="${prefix}robotiq_85_left_knuckle_joint" offset="0"/>
 		</joint>
-		<xacro:mimic_joint_plugin_gazebo name_prefix="${prefix}robotiq_85_right_inner_knuckle_joint"
+    <xacro:mimic_joint_plugin_gazebo name_prefix="${prefix}robotiq_85_right_inner_knuckle_joint"
 			parent_joint="${prefix}robotiq_85_left_knuckle_joint" mimic_joint="${prefix}robotiq_85_right_inner_knuckle_joint"
-			multiplier="1.0" max_effort="10.0" />
+      multiplier="1.0" max_effort="10.0" />
 		<link name="${prefix}robotiq_85_left_inner_knuckle_link">
 			<visual>
@@ -258,7 +248,7 @@
 			<mimic joint="${prefix}robotiq_85_left_knuckle_joint" multiplier="-1"/>
 		</joint>
-		<xacro:mimic_joint_plugin_gazebo name_prefix="${prefix}robotiq_85_left_finger_tip_joint"
+    <xacro:mimic_joint_plugin_gazebo name_prefix="${prefix}robotiq_85_left_finger_tip_joint"
 			parent_joint="${prefix}robotiq_85_left_knuckle_joint" mimic_joint="${prefix}robotiq_85_left_finger_tip_joint"
-			multiplier="1.0" max_effort="10.0" />
+      multiplier="1.0" max_effort="10.0" />
 		<joint name="${prefix}robotiq_85_right_finger_tip_joint" type="continuous">
 			<parent link="${prefix}robotiq_85_right_inner_knuckle_link"/>
@@ -269,7 +259,7 @@
 			<mimic joint="${prefix}robotiq_85_left_knuckle_joint" multiplier="-1"/>
 		</joint>
-		<xacro:mimic_joint_plugin_gazebo name_prefix="${prefix}robotiq_85_right_finger_tip_joint"
+    <xacro:mimic_joint_plugin_gazebo name_prefix="${prefix}robotiq_85_right_finger_tip_joint"
 			parent_joint="${prefix}robotiq_85_left_knuckle_joint" mimic_joint="${prefix}robotiq_85_right_finger_tip_joint"
-			multiplier="1.0" max_effort="10.0" />
+      multiplier="1.0" max_effort="10.0" />
 		<link name="${prefix}robotiq_85_left_finger_tip_link">
 			<visual>
